Commit message: Add RGB-D camera

File: my_robot/urdf/my_robot.xacro (robot description, xacro)
@@ -144,4 +144,12 @@
     <child link="camera" />
   </joint>
+  <!-- Add RGB-D camera -->
+  <joint name="camera_optical_joint" type="fixed">
+    <origin xyz="0 0 0" rpy="-1.5707 0 -1.5707"/>
+    <parent link="camera"/>
+    <child link="camera_link_optical"/>
+  </joint>
+  <link name="camera_link_optical">
+  </link>
   <!-- Add Lidar -->
   <link name="hokuyo">

Commit message: update launch files and robot configuration files

File: my_robot/urdf/my_robot.xacro (robot description, xacro)
@@ -146,5 +146,5 @@
   <!-- Add RGB-D camera -->
   <joint name="camera_optical_joint" type="fixed">
-    <origin xyz="0 0 0" rpy="-1.5707 0 -1.5707"/>
+    <origin xyz="0 0 0" rpy="0 0 0"/>
     <parent link="camera"/>
     <child link="camera_link_optical"/>
